File: design/gemini/pcb/gemini-panel/gemini-panel.kicad_pcb (KiCad board)
At the start: 2 copper layers, 250.2 x 84.2 mm, 149 parts

Commit message: add silkscreening, and layer visibility for model view
Parts:
- added L_G1: Logo_Gemini, Logo_Gemini, F.Cu at (58.8, -4.00)
- added R_G1: Logo_Gemini, Logo_Gemini, F.Cu at (-61.5, -4.00)
